Commit message: Combined launch and urdf fixes

File: urdf/jetank.xacro (robot description, xacro)
@@ -1,9 +1,9 @@
 <?xml version="1.0"?>
 <robot name="jetank" xmlns:xacro="http://www.ros.org/wiki/xacro">
-  <xacro:include filename="$(find robot_main)/urdf/properties.xacro"/>
-  <xacro:include filename="$(find robot_main)/urdf/jetank_wheel.xacro"/>
-  <xacro:include filename="$(find robot_main)/urdf/jetank_arm.xacro"/>
-  <xacro:include filename="$(find robot_main)/urdf/jetank_gripper.xacro"/>
-  <xacro:include filename="$(find robot_main)/urdf/jetank_camera.xacro"/>
+  <xacro:include filename="$(find jetank_ros2_main)/urdf/properties.xacro"/>
+  <xacro:include filename="$(find jetank_ros2_main)/urdf/jetank_wheel.xacro"/>
+  <xacro:include filename="$(find jetank_ros2_main)/urdf/jetank_arm.xacro"/>
+  <xacro:include filename="$(find jetank_ros2_main)/urdf/jetank_gripper.xacro"/>
+  <xacro:include filename="$(find jetank_ros2_main)/urdf/jetank_camera.xacro"/>
   <!-- Base link -->
   <link name="base_link" />

File: urdf/jetank_camera.xacro (robot description, xacro)
@@ -37,5 +37,5 @@
     <parent link="camera_base_plate_link"/>
     <child link="camera_left_link"/>
-    <origin xyz="${camera_heigth/2} ${camera_dist} ${0.0}" rpy="0 -1.57079632679 0"/>
+    <origin xyz="${camera_heigth/2} ${camera_dist} ${0.0}" rpy="0 -1.57079632679 3.14159265359"/>
   </joint>
   <!-- Camera right to base -->
@@ -43,5 +43,5 @@
     <parent link="camera_base_plate_link"/>
     <child link="camera_right_link"/>
-    <origin xyz="${camera_heigth/2} ${-camera_dist} ${0.0}" rpy="0 -1.57079632679 0"/>
+    <origin xyz="${camera_heigth/2} ${-camera_dist} ${0.0}" rpy="0 -1.57079632679 3.14159265359"/>
   </joint>
 </robot>
